File: electronique/PCB/R-IR.sch (KiCad schematic (older format))
At the start: 37 parts, among them J2 CONN_C1, J3 CONN_C3, J4 CONN_C2, J5 CONN_C4, U2 LM324

Commit message: new values
Parts:
- R6: value 22kR -> 330kR
Changed lines of the file:
@@
 P 4850 2750
 F 0 "R6" V 4930 2750 50  0000 C CNN
-F 1 "22kR" V 4850 2750 50  0000 C CNN
+F 1 "330kR" V 4850 2750 50  0000 C CNN
 F 2 "Discret:R4-LARGE_PADS" V 4780 2750 50  0001 C CNN
 F 3 "" H 4850 2750 50  0001 C CNN
