File: electronique/PCB/T-IR.sch (KiCad schematic (older format))
At the start: 5 parts, among them U3 NE555

Commit message: new values
Parts:
- C10: value 4,8nC -> 1nC
Changed lines of the file:
@@
 P 6550 3200
 F 0 "C10" H 6575 3300 50  0000 L CNN
-F 1 "4,8nC" H 6575 3100 50  0000 L CNN
+F 1 "1nC" H 6575 3100 50  0000 L CNN
 F 2 "Capacitors_THT:C_Rect_L7.0mm_W2.5mm_P5.00mm" H 6588 3050 50  0001 C CNN
 F 3 "" H 6550 3200 50  0001 C CNN
