File: electronique/PCB/uC-part.sch (KiCad schematic (older format))
At the start: 6 parts, among them U1 Arduino-nano, U5 trou-3, U6 trou-3, U7 trou-3

Commit message: new values
Parts:
- D1: symbol LED -> LED-RESCUE-Robot_sumo
Changed lines of the file:
@@
 $EndDescr
 $Comp
-L LED D1
+L LED-RESCUE-Robot_sumo D1
 U 1 1 5942F4DF
 P 3300 2300
+AR Path="/5942F4DF" Ref="D1"  Part="1"
+AR Path="/5942F2F4/5942F4DF" Ref="D1"  Part="1"
 F 0 "D1" H 3300 2400 50  0000 C CNN
 F 1 "LED_red" H 3300 2200 50  0000 C CNN
